Commit message: Lidar started

File: description/gazebo_control.xacro (robot description, xacro)
@@ -10,5 +10,5 @@
             <!-- Limits -->
             <max_wheel_torque>200</max_wheel_torque>
-            <max_wheel_acceleration>200</max_wheel_acceleration>
+            <max_wheel_acceleration>10.0</max_wheel_acceleration>
             <!-- Output -->
             <odometry_frame>odom</odometry_frame>

File: description/robot_core.xacro (robot description, xacro)
@@ -12,5 +12,8 @@
     </material>
     <material name="black">
-        <color rgba="0 0 0 1"/>
+        <color rgba=" 0 0 1"/>
+    </material>
+    <material name="red">
+        <color rgba="1 0 0 1"/>
     </material>
     <!-- BASE LINK -->
